File: hardware/pcb/radar-pcb.kicad_sch (KiCad schematic)
At the start: 66 parts, among them J1 Gniazdo DC 5,5/2,1 mm, srodek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, J10 Awaryjne wgrywanie: BOOT GND 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, J11 Piny DevKit J3 (kopia J3), J12 Piny DevKit J1 (kopia J2), J13 Listwa zasilania: GND 3V3 5V, J14 Pole prototypowe 1 (2x14, nie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, J15 Pole prototypowe 2 (2x14, nie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, J16 Pole prototypowe 3 (2x14, nie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, J17 Pole prototypowe 4 (2x14, nie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, J2 DevKit J1, J3 DevKit J3, J4 HC-SR04 (kabel): VCC TRIG ECH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, J5 Serwo SG90 (kabel): GND +5V S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, J6 MAX7219 Elegoo: VCC GND DIN C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, J7 OLED SH1106: VCC GND SCK SDA, J8 Buzzer: + -, J9 Przycisk zewnetrzny, Q2 2N3904 (TO-92, E B C), SW1 Przycisk ON/standby (katowy), U1 SN74AHCT125N (DIP-14)

Commit message: PCB v0.2: wszystkie listwy żeńskie (J4-J13)
Listwy J4, J5, J8, J9, J10, J11, J12 i J13 zmienione z goldpinów na gniazda żeńskie (ten sam rozstaw
i numeracja pinów, układ i trasowanie bez zmian). Lista zakupów i notatki zaktualizowane.
ERC 0 błędów; DRC 0 błędów, 0 niepołączonych, 0 niezgodności ze schematem. Nic nie sprawdzono na sprzęcie.

Co-Authored-By: Claude Sonnet 5.5 <noreply@anthropic.com>
Parts:
- J10, J5: footprint Connector_PinHeader_2.54mm:PinHeader_1x03_P2.54mm_Vertical -> Connector_PinSocket_2.54mm:PinSocket_1x03_P2.54mm_Vertical
- J11, J12: footprint Connector_PinHeader_2.54mm:PinHeader_1x16_P2.54mm_Vertical -> Connector_PinSocket_2.54mm:PinSocket_1x16_P2.54mm_Vertical
- J13: footprint Connector_PinHeader_2.54mm:PinHeader_1x08_P2.54mm_Vertical -> Connector_PinSocket_2.54mm:PinSocket_1x08_P2.54mm_Vertical
- J4: footprint Connector_PinHeader_2.54mm:PinHeader_1x04_P2.54mm_Vertical -> Connector_PinSocket_2.54mm:PinSocket_1x04_P2.54mm_Vertical
- J8, J9: footprint Connector_PinHeader_2.54mm:PinHeader_1x02_P2.54mm_Vertical -> Connector_PinSocket_2.54mm:PinSocket_1x02_P2.54mm_Vertical
